File: KiCad/openMicroInverter_dev/openMicroInverter_dev.sch (KiCad schematic (older format))
At the start: 92 parts, among them K1 ISLANDING RELAY, P1 CONN_01X02, P2 CONN_01X02, P3 ARDUINO_R3, Q1 N-CHANNEL, Q2 N-CHANNEL, Q3 N-CHANNEL, Q4 N-CHANNEL, Q5 Q_NPN_CBE, T1 LEM_LA55-P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

Commit message: Inverter1, measurements enabled
Parts:
- added LOGO1: Logo_Open_Hardware_Small, symbol Graphic:Logo_Open_Hardware_Small
- C10, C11, C12, C13, C15, C16, C17, C18: value C -> 100n
Connections:
- net GND: now also P3.29 (GND)
- net P5V0: no longer C6.1, U1.2 (BHI), U1.7 (AHI)
- net VREF_CP: now also C6.1
- net H_AHI: now reaches P3.18 (~~3)
- net H_AHI: now also U1.7 (AHI)
- net H_BHI: now reaches P3.26 (~~11)
- net H_BHI: now also U1.2 (BHI)
- net PLL_lock renamed PLL_LOCK
- net XOR_out renamed XOR_OUT
- no-connect marks 0 -> 10
Other:
- note added: "PLL loopfilter\n(obsolete)"
- note removed: "PLL loopfilter"
- moved on the sheet: C1, C2, D1, Q2, Q4, R14, R19, R26, R27, R4

Commit message: add new sketches, update docs
Parts:
- removed C20: 47uF, symbol openMicroInverter_dev-rescue:CP-SmartInverter_proto-rescue
- removed R33: 10K, symbol openMicroInverter_dev-rescue:R-SmartInverter_proto-rescue
- added RV1: 10k, symbol Device:R_POT_US
- C9: value 1n5 -> 10n
Connections:
- net Ibatt is gone; now on net Ibatt_scaled: P3.12 (AD3), R47.1
- net Iinv_ac is gone; now on net Iinv_scaled: P3.10 (AD1), R30.1
- net Vinv_ac is gone; now on net Vinv_scaled: P3.11 (AD2), R39.1
- net GND: now also RV1.3
- net Ibatt_scaled: no longer R46.2, R6.1, T1.3 (M)
- net Iinv_scaled: no longer R29.2, R8.1, T3.3 (M)
- net P5V0: now also RV1.1
- net Vinv_scaled: no longer R16.1, R38.2, T4.3 (M)
- net VPOT: now reaches P3.14 (AD5/SCL)
- net VPOT: now also RV1.2
- net VBATT+ renamed VDC+
- net Vbatt_scaled renamed Vdc_scaled
- net Vin_ac renamed Vgrid_scaled
- net Vline_scaled renamed Vgrid_sense
- net XOR_OUT renamed ZCD_OUT
- new net Ibatt_sense: R46.2, R6.1, T1.3 (M)
- new net Iinv_sense: R29.2, R8.1, T3.3 (M)
- new net Vinv_sense: R16.1, R38.2, T4.3 (M)
Other:
- note removed: "PLL loopfilter\n(obsolete)"
- moved on the sheet: C14, C19, C21, C22, C9, D2, R20, R22, R23, R24, R28, R30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
